File: monitor_osd_control/monitor_osd_control.kicad_pcb (KiCad board)
At the start: 2 copper layers, 50 x 58 mm, 21 parts, among them J1 Conn_01x09, J2 Conn_01x09, J3 Conn_01x05, J4 Conn_01x05, SW1 SW_Push, SW2 SW_Push, SW3 SW_Push, SW4 SW_Push, SW5 SW_Push, SW6 SW_Push, U1 TSSP58038

Commit message: 배선 최적화 및 pretty 경로 보정
Signed-off-by: Ju, Gyeong-min <jcmh74@gmail.com>
Parts:
- SW1, SW2, SW3, SW4, SW5: footprint monitor_control_board_library:SW_PUSH-12mm_Complex -> monitor_osd_control_library:SW_PUSH-12mm_Complex
Routing:
- net GND: track 170.3 -> 166.7 mm
Other:
- outline, holes or cut-outs redrawn
