File: monitor_osd_control/monitor_osd_control.kicad_sch (KiCad schematic)
At the start: 21 parts, among them J1 Conn_01x09, J2 Conn_01x09, J3 Conn_01x05, J4 Conn_01x05, SW1 SW_Push, SW2 SW_Push, SW3 SW_Push, SW4 SW_Push, SW5 SW_Push, SW6 SW_Push, U1 TSSP58038

Commit message: 캐패시터 크기 변경
Signed-off-by: Ju, Gyeong-min <jcmh74@gmail.com>
Parts:
- E1: footprint Capacitor_SMD:CP_Elec_4x5.4 -> Capacitor_SMD:CP_Elec_5x5.4
- SW1, SW2, SW3, SW4, SW5: footprint monitor_control_board_library:SW_PUSH-12mm_Complex -> monitor_osd_control_library:SW_PUSH-12mm_Complex
Changed lines of the file:
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@@
       (effects (font (size 1.27 1.27)))
     )
-    (property "Footprint" "monitor_control_board_library:SW_PUSH-12mm_Complex" (at 230.505 56.515 0)
+    (property "Footprint" "monitor_osd_control_library:SW_PUSH-12mm_Complex" (at 230.505 56.515 0)
       (effects (font (size 1.27 1.27)) hide)
     )
@@
       (effects (font (size 1.27 1.27)))
     )
-    (property "Footprint" "monitor_control_board_library:SW_PUSH-12mm_Complex" (at 208.28 56.515 0)
+    (property "Footprint" "monitor_osd_control_library:SW_PUSH-12mm_Complex" (at 208.28 56.515 0)
       (effects (font (size 1.27 1.27)) hide)
     )
@@
       (effects (font (size 1.27 1.27)))
     )
-    (property "Footprint" "monitor_control_board_library:SW_PUSH-12mm_Complex" (at 207.645 33.655 0)
+    (property "Footprint" "monitor_osd_control_library:SW_PUSH-12mm_Complex" (at 207.645 33.655 0)
       (effects (font (size 1.27 1.27)) hide)
     )
@@
       (effects (font (size 1.27 1.27)))
     )
-    (property "Footprint" "monitor_control_board_library:SW_PUSH-12mm_Complex" (at 208.28 80.01 0)
+    (property "Footprint" "monitor_osd_control_library:SW_PUSH-12mm_Complex" (at 208.28 80.01 0)
       (effects (font (size 1.27 1.27)) hide)
     )
@@
       (effects (font (size 1.27 1.27)))
     )
-    (property "Footprint" "monitor_control_board_library:SW_PUSH-12mm_Complex" (at 185.42 57.15 0)
+    (property "Footprint" "monitor_osd_control_library:SW_PUSH-12mm_Complex" (at 185.42 57.15 0)
       (effects (font (size 1.27 1.27)) hide)
     )
@@
       (effects (font (size 1.27 1.27)) (justify left))
     )
-    (property "Footprint" "Capacitor_SMD:CP_Elec_4x5.4" (at 114.3 160.655 0)
-      (effects (font (size 1.27 1.27)) hide)
-    )
+    (property "Footprint" "Capacitor_SMD:CP_Elec_5x5.4" (at 114.3 160.655 0)
+      (effects (font (size 1.27 1.27)) hide)
+    )
